Commit message: WIP: Tool grasping experiments.

File: assets/dexterity/tools/drill/black_and_decker_unknown/rigid.urdf (robot description, URDF)
Before this commit: robot rigid_drill, 1 links, 0 joints
Links:
- link base: geometry collision mesh filename=assets/downsampled_16k.obj; visual mesh filename=assets/downsampled_16k.obj
