Commit message: WIP: Tool grasping experiments.

File: assets/dexterity/tools/shelf/rigid.urdf (robot description, URDF)
Before this commit: robot shelf, 1 links, 0 joints
Links:
- link base_link: geometry collision box size=0.2 0.375 0.015; collision box size=0.2 0.375 0.15

Commit message: WIP: Tool grasping experiments.

File: assets/dexterity/tools/shelf/rigid.urdf (robot description, URDF)
Before this commit: robot shelf, 1 links, 0 joints
Links:
- link base_link: geometry collision box size=0.2 0.375 0.018; collision box size=0.2 0.375 0.15
