Commit message: WIP: Tool grasping experiments.

File: assets/dexterity/tools/drill/blank_hagen_unknown/site.urdf (robot description, URDF)
Before this commit: robot drill, 4 links, 3 joints
Links:
- removed link bit
- removed link chuck
- removed link trigger
- link base: geometry visual mesh filename=assets/downsampled_16k.obj
Joints:
- removed joint base_to_chuck
- removed joint base_to_trigger
- removed joint chuck_to_bit

File: assets/dexterity/tools/drill/drill_and_driver_l76/rigid.urdf (robot description, URDF)
Before this commit: robot site, 1 links, 0 joints
Links:
- link base: geometry collision mesh filename=assets/downsampled_16k.obj; visual mesh filename=assets/downsampled_16k.obj
