Commit message: Adjust weights of YCB objects.

File: assets/dexterity/object_sets/urdf/ycb/002_master_chef_can.urdf (robot description, URDF)
Before this commit: robot 002_master_chef_can, 1 links, 0 joints
Links:
- link base_link: mass 0.325 -> 0.067

File: assets/dexterity/object_sets/urdf/ycb/003_cracker_box.urdf (robot description, URDF)
Before this commit: robot 003_cracker_box, 1 links, 0 joints
Links:
- link base_link: mass 0.36 -> 0.066

File: assets/dexterity/object_sets/urdf/ycb/004_sugar_box.urdf (robot description, URDF)
Before this commit: robot 004_sugar_box, 1 links, 0 joints
Links:
- link base_link: mass 0.46 -> 0.035

File: assets/dexterity/object_sets/urdf/ycb/005_tomato_soup_can.urdf (robot description, URDF)
Before this commit: robot 005_tomato_soup_can, 1 links, 0 joints
Links:
- link base_link: mass 0.2 -> 0.037

File: assets/dexterity/object_sets/urdf/ycb/006_mustard_bottle.urdf (robot description, URDF)
Before this commit: robot 006_mustard_bottle, 1 links, 0 joints
Links:
- link base_link: mass 0.58 -> 0.045

File: assets/dexterity/object_sets/urdf/ycb/007_tuna_fish_can.urdf (robot description, URDF)
Before this commit: robot 007_tuna_fish_can, 1 links, 0 joints
Links:
- link base_link: mass 0.16 -> 0.023

File: assets/dexterity/object_sets/urdf/ycb/008_pudding_box.urdf (robot description, URDF)
Before this commit: robot 008_pudding_box, 1 links, 0 joints
Links:
- link base_link: mass 0.18 -> 0.024

File: assets/dexterity/object_sets/urdf/ycb/009_gelatin_box.urdf (robot description, URDF)
Before this commit: robot 009_gelatin_box, 1 links, 0 joints
Links:
- link base_link: mass 0.095 -> 0.031

File: assets/dexterity/object_sets/urdf/ycb/010_potted_meat_can.urdf (robot description, URDF)
Before this commit: robot 010_potted_meat_can, 1 links, 0 joints
Links:
- link base_link: mass 0.36 -> 0.023

File: assets/dexterity/object_sets/urdf/ycb/011_banana.urdf (robot description, URDF)
Before this commit: robot 011_banana, 1 links, 0 joints
Links:
- link base_link: mass 0.12 -> 0.061

File: assets/dexterity/object_sets/urdf/ycb/012_strawberry.urdf (robot description, URDF)
Before this commit: robot 012_strawberry, 1 links, 0 joints
Links:
- link base_link: mass 0.02 -> 0.017

File: assets/dexterity/object_sets/urdf/ycb/013_apple.urdf (robot description, URDF)
Before this commit: robot 013_apple, 1 links, 0 joints
Links:
- link base_link: mass 0.1 -> 0.063

File: assets/dexterity/object_sets/urdf/ycb/014_lemon.urdf (robot description, URDF)
Before this commit: robot 014_lemon, 1 links, 0 joints
Links:
- link base_link: mass 0.08 -> 0.034

File: assets/dexterity/object_sets/urdf/ycb/015_peach.urdf (robot description, URDF)
Before this commit: robot 015_peach, 1 links, 0 joints
Links:
- link base_link: mass 0.08 -> 0.033

File: assets/dexterity/object_sets/urdf/ycb/016_pear.urdf (robot description, URDF)
Before this commit: robot 016_pear, 1 links, 0 joints
Links:
- link base_link: mass 0.1 -> 0.049

File: assets/dexterity/object_sets/urdf/ycb/017_orange.urdf (robot description, URDF)
Before this commit: robot 017_orange, 1 links, 0 joints
Links:
- link base_link: mass 0.09 -> 0.051

File: assets/dexterity/object_sets/urdf/ycb/018_plum.urdf (robot description, URDF)
Before this commit: robot 018_plum, 1 links, 0 joints
Links:
- link base_link: mass 0.05 -> 0.026

File: assets/dexterity/object_sets/urdf/ycb/021_bleach_cleanser.urdf (robot description, URDF)
Before this commit: robot 021_bleach_cleanser, 1 links, 0 joints
Links:
- link base_link: mass 1.05 -> 0.054

File: assets/dexterity/object_sets/urdf/ycb/024_bowl.urdf (robot description, URDF)
Before this commit: robot 024_bowl, 1 links, 0 joints
Links:
- link base_link: mass 0.18 -> 0.131

File: assets/dexterity/object_sets/urdf/ycb/025_mug.urdf (robot description, URDF)
Before this commit: robot 025_mug, 1 links, 0 joints
Links:
- link base_link: mass 0.17 -> 0.098
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